File: tests/XMOStests/tests.sch (KiCad schematic (older format))
At the start: 2 parts, among them U1 XS1-L1-128, U3 XS1-L1-64

Commit message: Updated after repos split.
Parts:
- removed U3: XS1-L1-64, symbol XS1-L1-64
- added U2: XS1-L1-64, symbol XS1-L1-64
Changed lines of the file:
@@
-EESchema Schematic File Version 2  date Tue 05 Apr 2011 10:59:55 AM PDT
+EESchema Schematic File Version 2  date Tue 05 Apr 2011 01:14:58 PM PDT
+LIBS:XS1-L1-64
+LIBS:XS1-L1-128
 LIBS:power
 LIBS:device
@@
 LIBS:contrib
 LIBS:valves
-LIBS:XS1-L1-64
-LIBS:XS1-L1-128
 LIBS:tests-cache
 EELAYER 24  0
@@
 $EndDescr
 $Comp
-L XS1-L1-128 U?
-U 5 1 4D9B5367
-P 4800 6150
-AR Path="/4D9B5146" Ref="U?"  Part="4"
-AR Path="/4D9B5367" Ref="U1"  Part="5"
-F 0 "U1" H 4800 7450 50  0000 C CNN
-F 1 "XS1-L1-128" H 4800 7350 50  0000 C CNN
-	5    4800 6150
+L XS1-L1-128 U1
+U 5 1 4D9B782B
+P 5150 6050
+F 0 "U1" H 5150 7350 50  0000 C CNN
+F 1 "XS1-L1-128" H 5150 7250 50  0000 C CNN
+	5    5150 6050
+	1    0    0    -1
+$EndComp
+$Comp
+L XS1-L1-128 U1
+U 4 1 4D9B7779
+P 3600 6250
+F 0 "U1" H 3600 7550 50  0000 C CNN
+F 1 "XS1-L1-128" H 3600 7450 50  0000 C CNN
+	4    3600 6250
+	1    0    0    -1
+$EndComp
+$Comp
+L XS1-L1-128 U1
+U 3 1 4D9B776C
+P 2050 5400
+F 0 "U1" H 2050 6700 50  0000 C CNN
+F 1 "XS1-L1-128" H 2050 6600 50  0000 C CNN
+	3    2050 5400
+	1    0    0    -1
+$EndComp
+$Comp
+L XS1-L1-128 U1
+U 2 1 4D9B7761
+P 2200 3200
+F 0 "U1" H 2200 4500 50  0000 C CNN
+F 1 "XS1-L1-128" H 2200 4400 50  0000 C CNN
+	2    2200 3200
+	1    0    0    -1
+$EndComp
+$Comp
+L XS1-L1-128 U1
+U 1 1 4D9B7749
+P 4800 2900
+F 0 "U1" H 4800 4200 50  0000 C CNN
+F 1 "XS1-L1-128" H 4800 4100 50  0000 C CNN
+	1    4800 2900
+	1    0    0    -1
+$EndComp
+$Comp
+L XS1-L1-64 U2
+U 3 1 4D9B771E
+P 9850 4000
+F 0 "U2" H 9050 4800 50  0000 C CNN
+F 1 "XS1-L1-64" H 9050 4900 50  0000 C CNN
+	3    9850 4000
+	1    0    0    -1
+$EndComp
+$Comp
+L XS1-L1-64 U2
+U 2 1 4D9B7706
+P 7850 5250
+F 0 "U2" H 7050 6050 50  0000 C CNN
+F 1 "XS1-L1-64" H 7050 6150 50  0000 C CNN
+	2    7850 5250
+	1    0    0    -1
+$EndComp
+$Comp
+L XS1-L1-64 U2
+U 1 1 4D9B76F2
+P 7750 2850
+F 0 "U2" H 6950 3650 50  0000 C CNN
+F 1 "XS1-L1-64" H 6950 3750 50  0000 C CNN
+	1    7750 2850
 	1    0    0    -1
 $EndComp
@@
 Text Notes 2800 1350 0    60   ~ 0
 XS1-L1-128 - in Five sub-parts
-$Comp
-L XS1-L1-64 U3
-U 3 1 4D9B518F
-P 10100 3850
-F 0 "U3" H 9300 4650 50  0000 C CNN
-F 1 "XS1-L1-64" H 9300 4750 50  0000 C CNN
-	3    10100 3850
-	1    0    0    -1
-$EndComp
-$Comp
-L XS1-L1-64 U3
-U 2 1 4D9B5175
-P 7950 5100
-F 0 "U3" H 7150 5900 50  0000 C CNN
-F 1 "XS1-L1-64" H 7150 6000 50  0000 C CNN
-	2    7950 5100
-	1    0    0    -1
-$EndComp
-$Comp
-L XS1-L1-64 U3
-U 1 1 4D9B5169
-P 7900 2750
-F 0 "U3" H 7100 3550 50  0000 C CNN
-F 1 "XS1-L1-64" H 7100 3650 50  0000 C CNN
-	1    7900 2750
-	1    0    0    -1
-$EndComp
-$Comp
-L XS1-L1-128 U1
-U 4 1 4D9B5146
-P 3600 6300
-F 0 "U1" H 3600 7600 50  0000 C CNN
-F 1 "XS1-L1-128" H 3600 7500 50  0000 C CNN
-	4    3600 6300
-	1    0    0    -1
-$EndComp
-$Comp
-L XS1-L1-128 U1
-U 3 1 4D9B5136
-P 2200 5450
-F 0 "U1" H 2200 6750 50  0000 C CNN
-F 1 "XS1-L1-128" H 2200 6650 50  0000 C CNN
-	3    2200 5450
-	1    0    0    -1
-$EndComp
-$Comp
-L XS1-L1-128 U1
-U 2 1 4D9B50E5
-P 2500 3250
-F 0 "U1" H 2500 4550 50  0000 C CNN
-F 1 "XS1-L1-128" H 2500 4450 50  0000 C CNN
-	2    2500 3250
-	1    0    0    -1
-$EndComp
-$Comp
-L XS1-L1-128 U1
-U 1 1 4D9B50D7
-P 4550 2950
-F 0 "U1" H 4550 4250 50  0000 C CNN
-F 1 "XS1-L1-128" H 4550 4150 50  0000 C CNN
-	1    4550 2950
-	1    0    0    -1
-$EndComp
 $EndSCHEMATC
